File: Hardware/DOC-00001.brd (EAGLE design)
At the start: 25.4 x 12.7 mm, 8 parts

Commit message: Added BOM.
Parts:
- U$1: value MCP3021XX-X/OT -> MCP3021A0T-E/OT
- U$2: value MCP3021XX-X/OT -> MCP3021A1T-E/OT
- U$3: value MCP3021XX-X/OT -> MCP3021A2T-E/OT
- U$4: value MCP3021XX-X/OT -> MCP3021A3T-E/OT
Changed lines of the file:
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@@
 </autorouter>
 <elements>
-<element name="U$1" library="MCP3021AX" package="SOT-23-5_MC" value="MCP3021XX-X/OT" x="5.0292" y="8.255" rot="R270"/>
-<element name="U$2" library="MCP3021AX" package="SOT-23-5_MC" value="MCP3021XX-X/OT" x="12.446" y="8.255" rot="R270"/>
-<element name="U$3" library="MCP3021AX" package="SOT-23-5_MC" value="MCP3021XX-X/OT" x="17.8308" y="8.255" rot="R270"/>
-<element name="U$4" library="MCP3021AX" package="SOT-23-5_MC" value="MCP3021XX-X/OT" x="23.2156" y="8.255" rot="R270"/>
-<element name="R1" library="resistor" package="R0805" value="4.7k" x="2.032" y="8.128" smashed="yes" rot="MR0"/>
-<element name="R2" library="resistor" package="R0805" value="4.7k" x="2.032" y="4.318" smashed="yes" rot="MR0"/>
-<element name="C1" library="resistor" package="C0805K" value="0.1uF" x="2.286" y="11.43" smashed="yes" rot="MR0"/>
-<element name="JP1" library="pinhead" package="1X08" value="v" x="13.716" y="2.032" smashed="yes"/>
+<element name="U$1" library="MCP3021AX" package="SOT-23-5_MC" value="MCP3021A0T-E/OT " x="5.0292" y="8.255" rot="R270">
+<attribute name="MPN" value="MCP3021A0T-E/OT" x="5.0292" y="8.255" size="1.778" layer="27" rot="R270" display="off"/>
+<attribute name="PRICE" value="1.07" x="5.0292" y="8.255" size="1.778" layer="27" rot="R270" display="off"/>
+<attribute name="STORE" value="microchipdirect.com" x="5.0292" y="8.255" size="1.778" layer="27" rot="R270" display="off"/>
+</element>
+<element name="U$2" library="MCP3021AX" package="SOT-23-5_MC" value="MCP3021A1T-E/OT " x="12.446" y="8.255" rot="R270">
+<attribute name="MPN" value="MCP3021A1T-E/OT" x="12.446" y="8.255" size="1.778" layer="27" rot="R270" display="off"/>
+<attribute name="PRICE" value="1.07" x="12.446" y="8.255" size="1.778" layer="27" rot="R270" display="off"/>
+<attribute name="STORE" value="microchipdirect.com" x="12.446" y="8.255" size="1.778" layer="27" rot="R270" display="off"/>
+</element>
+<element name="U$3" library="MCP3021AX" package="SOT-23-5_MC" value="MCP3021A2T-E/OT " x="17.8308" y="8.255" rot="R270">
+<attribute name="MPN" value="MCP3021A2T-E/OT" x="17.8308" y="8.255" size="1.778" layer="27" rot="R270" display="off"/>
+<attribute name="PRICE" value="1.07" x="17.8308" y="8.255" size="1.778" layer="27" rot="R270" display="off"/>
+<attribute name="STORE" value="microchipdirect.com" x="17.8308" y="8.255" size="1.778" layer="27" rot="R270" display="off"/>
+</element>
+<element name="U$4" library="MCP3021AX" package="SOT-23-5_MC" value="MCP3021A3T-E/OT " x="23.2156" y="8.255" rot="R270">
+<attribute name="MPN" value="MCP3021A3T-E/OT" x="23.2156" y="8.255" size="1.778" layer="27" rot="R270" display="off"/>
+<attribute name="PRICE" value="1.07" x="23.2156" y="8.255" size="1.778" layer="27" rot="R270" display="off"/>
+<attribute name="STORE" value="microchipdirect.com" x="23.2156" y="8.255" size="1.778" layer="27" rot="R270" display="off"/>
+</element>
+<element name="R1" library="resistor" package="R0805" value="4.7k" x="2.032" y="8.128" smashed="yes" rot="MR0">
+<attribute name="MPN" value="CRCW08054K70FKEA" x="2.032" y="8.128" size="1.778" layer="28" rot="MR0" display="off"/>
+<attribute name="PRICE" value="0.08" x="2.032" y="8.128" size="1.778" layer="28" rot="MR0" display="off"/>
+<attribute name="STORE" value="mouser.com" x="2.032" y="8.128" size="1.778" layer="28" rot="MR0" display="off"/>
+</element>
+<element name="R2" library="resistor" package="R0805" value="4.7k" x="2.032" y="4.318" smashed="yes" rot="MR0">
+<attribute name="MPN" value="CRCW08054K70FKEA" x="2.032" y="4.318" size="1.778" layer="28" rot="MR0" display="off"/>
+<attribute name="PRICE" value="0.08" x="2.032" y="4.318" size="1.778" layer="28" rot="MR0" display="off"/>
+<attribute name="STORE" value="mouser.com" x="2.032" y="4.318" size="1.778" layer="28" rot="MR0" display="off"/>
+</element>
+<element name="C1" library="resistor" package="C0805K" value="0.1uF" x="2.286" y="11.43" smashed="yes" rot="MR0">
+<attribute name="MPN" value="VJ0805Y104MXXAC" x="2.286" y="11.43" size="1.778" layer="28" rot="MR0" display="off"/>
+<attribute name="PRICE" value="0.06" x="2.286" y="11.43" size="1.778" layer="28" rot="MR0" display="off"/>
+<attribute name="STORE" value="mouser.com" x="2.286" y="11.43" size="1.778" layer="28" rot="MR0" display="off"/>
+</element>
+<element name="JP1" library="pinhead" package="1X08" value="v" x="13.716" y="2.032" smashed="yes">
+<attribute name="MPN" value="825433-8" x="13.716" y="2.032" size="1.778" layer="27" display="off"/>
+<attribute name="PRICE" value="0.84" x="13.716" y="2.032" size="1.778" layer="27" display="off"/>
+<attribute name="STORE" value="mouser.com" x="13.716" y="2.032" size="1.778" layer="27" display="off"/>
+</element>
 </elements>
 <signals>
